Commit message: code running but figure out frames

File: urdf/camera_setup.urdf.xacro (robot description, xacro)
@@ -11,10 +11,10 @@
   <xacro:arg name="camera_frame" default="camera_link"/> -->
   <!-- Define properties to make expressions safer and debuggable -->
-  <xacro:property name="camera_x" value="0.0"/>
-  <xacro:property name="camera_y" value="0.0"/>
-  <xacro:property name="camera_z" value="0.1"/>
-  <xacro:property name="camera_roll" value="0.0"/>
+  <xacro:property name="camera_x" value="0.01"/>
+  <xacro:property name="camera_y" value="0.02"/>
+  <xacro:property name="camera_z" value="0.03"/>
+  <xacro:property name="camera_roll" value="-1.57"/>
   <xacro:property name="camera_pitch" value="0.0"/>
-  <xacro:property name="camera_yaw" value="0.0"/>
+  <xacro:property name="camera_yaw" value="-1.57"/>
   <!-- Include the dummy robot URDF -->
   <xacro:include filename="$(find board_calib)/urdf/robot_description.urdf.xacro"/>
@@ -30,7 +30,9 @@
   <link name="charuco_board_link"/>
   <joint name="base_to_charuco_board_joint" type="fixed">
-    <parent link="map"/>
+    <parent link="base_link"/>
     <child link="charuco_board_link"/>
-    <origin xyz="0.27 0 0.1" rpy="0 0 0"/> <!-- update these values to match your setup -->
+    <origin xyz="0.25 0.08 -0.03" rpy="1.57 0.0 -1.57"/> <!-- update these values to match your setup -->
   </joint>
+  <!-- Tranform between camera frame and camera optical frame -->
+  <!-- xyz="0 0 0" rpy="-1.57 0.0 -1.57"-->
 </robot>

File: urdf/robot_description.urdf.xacro (robot description, xacro)
@@ -14,5 +14,5 @@
     <parent link="base_link"/>
     <child link="head_link"/>
-    <origin xyz="0 0 0.13" rpy="0 0 0"/>
+    <origin xyz="0 0 0.23" rpy="0 0 0"/>
   </joint>
 </robot>

Commit message: working perfectly, static calibration, 1 sample, 1 camera

File: urdf/camera_setup.urdf.xacro (robot description, xacro)
@@ -11,20 +11,20 @@
   <xacro:arg name="camera_frame" default="camera_link"/> -->
   <!-- Define properties to make expressions safer and debuggable -->
-  <xacro:property name="camera_x" value="0.01"/>
-  <xacro:property name="camera_y" value="0.02"/>
-  <xacro:property name="camera_z" value="0.03"/>
-  <xacro:property name="camera_roll" value="-1.57"/>
+  <xacro:property name="camera_x" value="0.00"/>
+  <xacro:property name="camera_y" value="0.00"/>
+  <xacro:property name="camera_z" value="0.15"/>
+  <xacro:property name="camera_roll" value="0.0"/>
   <xacro:property name="camera_pitch" value="0.0"/>
-  <xacro:property name="camera_yaw" value="-1.57"/>
+  <xacro:property name="camera_yaw" value="0.0"/>
   <!-- Include the dummy robot URDF -->
   <xacro:include filename="$(find board_calib)/urdf/robot_description.urdf.xacro"/>
   <!-- Camera link -->
-  <link name="camera_link"/>
+  <!-- <link name="camera_link"/> -->
   <!-- Mount camera to robot base -->
-  <joint name="base_to_camera_joint" type="fixed">
+  <!-- <joint name="base_to_camera_joint" type="fixed">
     <parent link="base_link"/>
     <child link="camera_link"/>
     <origin xyz="${camera_x} ${camera_y} ${camera_z}" rpy="${camera_roll} ${camera_pitch} ${camera_yaw}"/>
-  </joint>
+  </joint> -->
   <!-- Charuco board fixed in front of base_link, adjust as per your setup -->
   <link name="charuco_board_link"/>
@@ -32,5 +32,5 @@
     <parent link="base_link"/>
     <child link="charuco_board_link"/>
-    <origin xyz="0.25 0.08 -0.03" rpy="1.57 0.0 -1.57"/> <!-- update these values to match your setup -->
+    <origin xyz="-0.06 0.22 0.015" rpy="1.57 0.0 0.0"/> <!-- update these values to match your setup -->
   </joint>
   <!-- Tranform between camera frame and camera optical frame -->

File: urdf/robot_description.urdf.xacro (robot description, xacro)
@@ -7,12 +7,13 @@
     <parent link="map"/>
     <child link="base_link"/>
-    <origin xyz="0.0 0.0 0.07" rpy="0 0 0"/>
+    <origin xyz="0.1 0.1 0.1" rpy="0 0 0"/>
   </joint>
   <!-- base link to head link -->
+  <!-- <link name="base_link"/> -->
   <link name="head_link"/>
   <joint name="base_to_head_joint" type="fixed">
     <parent link="base_link"/>
     <child link="head_link"/>
-    <origin xyz="0 0 0.23" rpy="0 0 0"/>
+    <origin xyz="0 0 0.2" rpy="0 0 0"/>
   </joint>
 </robot>

Commit message: urdf updated

File: urdf/camera_setup.urdf.xacro (robot description, xacro)
@@ -32,5 +32,5 @@
     <parent link="base_link"/>
     <child link="charuco_board_link"/>
-    <origin xyz="-0.06 0.22 0.015" rpy="1.57 0.0 0.0"/> <!-- update these values to match your setup -->
+    <origin xyz="-0.055 0.170 0.010" rpy="1.57 0.0 0.0"/> <!-- update these values to match your setup -->
   </joint>
   <!-- Tranform between camera frame and camera optical frame -->

File: urdf/robot_description.urdf.xacro (robot description, xacro)
@@ -7,5 +7,5 @@
     <parent link="map"/>
     <child link="base_link"/>
-    <origin xyz="0.1 0.1 0.1" rpy="0 0 0"/>
+    <origin xyz="0.00 0.15 0.00" rpy="0 0 0"/>
   </joint>
   <!-- base link to head link -->
@@ -15,5 +15,5 @@
     <parent link="base_link"/>
     <child link="head_link"/>
-    <origin xyz="0 0 0.2" rpy="0 0 0"/>
+    <origin xyz="0.00 0.00 0.20" rpy="0 0 0"/>
   </joint>
 </robot>

Commit message: Fetching TF correctly from Robot TF

File: urdf/camera_setup.urdf.xacro (robot description, xacro)
@@ -11,12 +11,12 @@
   <xacro:arg name="camera_frame" default="camera_link"/> -->
   <!-- Define properties to make expressions safer and debuggable -->
-  <xacro:property name="camera_x" value="0.00"/>
+  <!-- <xacro:property name="camera_x" value="0.00"/>
   <xacro:property name="camera_y" value="0.00"/>
   <xacro:property name="camera_z" value="0.15"/>
   <xacro:property name="camera_roll" value="0.0"/>
   <xacro:property name="camera_pitch" value="0.0"/>
-  <xacro:property name="camera_yaw" value="0.0"/>
-  <!-- Include the dummy robot URDF -->
-  <xacro:include filename="$(find board_calib)/urdf/robot_description.urdf.xacro"/>
+  <xacro:property name="camera_yaw" value="0.0"/> -->
+  <!-- Include the Robot URDF -->
+  <!-- <xacro:include filename="$(find board_calib)/urdf/robot_description.urdf.xacro"/> -->
   <!-- Camera link -->
   <!-- <link name="camera_link"/> -->
@@ -27,10 +27,40 @@
     <origin xyz="${camera_x} ${camera_y} ${camera_z}" rpy="${camera_roll} ${camera_pitch} ${camera_yaw}"/>
   </joint> -->
-  <!-- Charuco board fixed in front of base_link, adjust as per your setup -->
+  <!-- Attach to Global Map -->
+  <link name="map"/>
+  <link name="calibration_map"/>
+  <joint name="map_to_calibration_map" type="fixed">
+    <parent link="map"/>
+    <child link="calibration_map"/>
+    <origin xyz="0 0 0" rpy="0.0 0.0 0.0"/>
+  </joint>
+  <!-- CALIBRATION BOARD & RELATED LINKS-->
+  <!-- Map to Table Link -->
+  <link name="table_link"/>
+  <joint name="calibration_map_to_table_link" type="fixed">
+    <parent link="calibration_map"/>
+    <child link="table_link"/>
+    <origin xyz="0.755 0.500 0.397" rpy="0.0 0.0 0.0"/>
+  </joint>
+  <!-- Map to Charuco Board Centre Link -->
+  <link name="charuco_board_centre_link"/>
+  <joint name="map_to_charuco_board" type="fixed">
+    <parent link="calibration_map"/>
+    <child link="charuco_board_centre_link"/>
+    <!-- update these values to match your setup -->
+    <!-- Desk Setup -->
+    <origin xyz="0.00 0.20 0.065" rpy="1.57 0.0 0.0"/>
+    <!-- UR Setup -->
+    <!-- Towards Arms -->
+    <!-- <origin xyz="0.325 0.0 0.407" rpy="0.0 0.0 -1.57"/> -->
+    <!-- Towards Door -->
+    <!-- <origin xyz="0.685 0.0 0.407" rpy="0.0 0.0 -1.57"/> -->
+  </joint>
+  <!-- Charuco Board Centre Link to Charuco Board Link -->
   <link name="charuco_board_link"/>
-  <joint name="base_to_charuco_board_joint" type="fixed">
-    <parent link="base_link"/>
+  <joint name="charuco_board_centre_to_charuco_board" type="fixed">
+    <parent link="charuco_board_centre_link"/>
     <child link="charuco_board_link"/>
-    <origin xyz="-0.055 0.170 0.010" rpy="1.57 0.0 0.0"/> <!-- update these values to match your setup -->
+    <origin xyz="-0.065 -0.065 0.0" rpy="0.0 0.0 0.0"/> <!-- update these values to match your setup -->
   </joint>
   <!-- Tranform between camera frame and camera optical frame -->
